File: Electronique/Carte Arduino/Carte Arduino.sch (KiCad schematic (older format))
At the start: 8 parts

Commit message: Electronique/Carte Arduino/Carte Arduino.sch : - Ajout des composants I²C (Gyroscope, Acceleromètre, Humidité)
Parts:
- added P?: CONN_4, symbol CONN_4
- added P? (x2): CONN_8, symbol CONN_8
Connections:
- net labels added: Arduino - SCL, Arduino - SDA, GND
- wire segments 12 -> 32
- no-connect marks 0 -> 4
Other:
- note added: "Accelerometre"
- note added: "Capteur Humidite"
- note added: "Capteur pression exterieure"
- note added: "Capteur pression interieure"
- note added: "Capteur temperature exterieure"
- note added: "Capteur temperature interieure"
- note added: "Gyroscope"
Changed lines of the file:
@@
-EESchema Schematic File Version 1
-LIBS:power,device,conn,linear,regul,74xx,cmos4000,adc-dac,memory,xilinx,special,microcontrollers,dsp,microchip,analog_switches,motorola,texas,intel,audio,interface,digital-audio,philips,display,cypress,siliconi,contrib,valves
+EESchema Schematic File Version 2  date 10/12/2011 16:53:54
+LIBS:power
+LIBS:device
+LIBS:transistors
+LIBS:conn
+LIBS:linear
+LIBS:regul
+LIBS:74xx
+LIBS:cmos4000
+LIBS:adc-dac
+LIBS:memory
+LIBS:xilinx
+LIBS:special
+LIBS:microcontrollers
+LIBS:dsp
+LIBS:microchip
+LIBS:analog_switches
+LIBS:motorola
+LIBS:texas
+LIBS:intel
+LIBS:audio
+LIBS:interface
+LIBS:digital-audio
+LIBS:philips
+LIBS:display
+LIBS:cypress
+LIBS:siliconi
+LIBS:opto
+LIBS:atmel
+LIBS:contrib
+LIBS:valves
+LIBS:Carte Arduino-cache
 EELAYER 23  0
 EELAYER END
 $Descr A4 11700 8267
+encoding utf-8
 Sheet 1 1
 Title ""
-Date "9 dec 2011"
+Date "10 dec 2011"
 Rev ""
 Comp ""
@@
 Comment4 ""
 $EndDescr
+Text Notes 1850 4200 1    60   ~ 0
+Capteur temperature exterieure
+Text Notes 2250 4200 1    60   ~ 0
+Capteur pression exterieure
+Text Notes 1450 4200 1    60   ~ 0
+Capteur pression interieure
+Text Notes 1050 4200 1    60   ~ 0
+Capteur temperature interieure
+Text Notes 5600 5850 0    60   ~ 0
+Accelerometre
+Wire Wire Line
+	6300 6400 6300 6500
+Wire Wire Line
+	6200 6400 6200 6500
+Wire Wire Line
+	6000 6400 6000 6500
+Wire Wire Line
+	5800 6400 5800 6500
+Wire Wire Line
+	5600 6400 5600 6500
+Wire Wire Line
+	5200 6400 5200 6500
+Wire Wire Line
+	5000 6400 5000 6500
+Wire Wire Line
+	4800 6400 4800 6500
+Wire Wire Line
+	4600 6400 4600 6500
+Wire Wire Line
+	4200 6400 4200 6500
+Wire Wire Line
+	4000 6400 4000 6500
+Wire Wire Line
+	900  5350 900  5500
+Wire Wire Line
+	900  4750 900  4850
+Wire Wire Line
+	1100 4850 1100 4750
+Wire Wire Line
+	1500 4850 1500 4750
+Wire Wire Line
+	1300 4750 1300 4850
+Wire Wire Line
+	1300 5350 1300 5500
+Wire Wire Line
+	1700 5350 1700 5500
+Wire Wire Line
+	1700 4750 1700 4850
+Wire Wire Line
+	1900 4850 1900 4750
+Wire Wire Line
+	2300 4850 2300 4750
+Wire Wire Line
+	2100 4750 2100 4850
 Wire Wire Line
 	2100 5350 2100 5500
 Wire Wire Line
-	2100 4750 2100 4850
-Wire Wire Line
-	2300 4850 2300 4750
-Wire Wire Line
-	1900 4850 1900 4750
-Wire Wire Line
-	1700 4750 1700 4850
-Wire Wire Line
-	1700 5350 1700 5500
+	4100 6400 4100 6500
+Wire Wire Line
+	4300 6400 4300 6500
+Wire Wire Line
+	4700 6400 4700 6500
+Wire Wire Line
+	4900 6400 4900 6500
+Wire Wire Line
+	5100 6400 5100 6500
+Wire Wire Line
+	5300 6400 5300 6500
+Wire Wire Line
+	5700 6400 5700 6500
+Wire Wire Line
+	5900 6400 5900 6500
+Wire Wire Line
+	6100 6400 6100 6500
+$Comp
+L CONN_8 P?
+U 1 1 4EE37ED4
+P 5950 6050
+F 0 "P?" V 5900 6050 60  0000 C CNN
+F 1 "CONN_8" V 6000 6050 60  0000 C CNN
+	1    5950 6050
+	0    -1   -1   0
+$EndComp
+Text Notes 4700 5850 0    60   ~ 0
+Gyroscope
+Text Notes 3650 5850 0    60   ~ 0
+Capteur Humidite
+NoConn ~ 5200 6500
+NoConn ~ 5100 6500
+$Comp
+L GND #PWR?
+U 1 1 4EE37BF2
+P 5300 6500
+F 0 "#PWR?" H 5300 6500 30  0001 C CNN
+F 1 "GND" H 5300 6430 30  0001 C CNN
+	1    5300 6500
+	1    0    0    -1
+$EndComp
+NoConn ~ 5000 6500
+NoConn ~ 4900 6500
+Text Label 4800 6500 3    60   ~ 0
+Arduino - SDA
+Text Label 4700 6500 3    60   ~ 0
+Arduino - SCL
+$Comp
+L +5V #PWR?
+U 1 1 4EE37B76
+P 4600 6500
+F 0 "#PWR?" H 4600 6590 20  0001 C CNN
+F 1 "+5V" H 4600 6590 30  0000 C CNN
+	1    4600 6500
+	-1   0    0    1
+$EndComp
+$Comp
+L CONN_8 P?
+U 1 1 4EE37B01
+P 4950 6050
+F 0 "P?" V 4900 6050 60  0000 C CNN
+F 1 "CONN_8" V 5000 6050 60  0000 C CNN
+	1    4950 6050
+	0    -1   -1   0
+$EndComp
+$Comp
+L GND #PWR?
+U 1 1 4EE3788C
+P 4100 6500
+F 0 "#PWR?" H 4100 6500 30  0001 C CNN
+F 1 "GND" H 4100 6430 30  0001 C CNN
+	1    4100 6500
+	1    0    0    -1
+$EndComp
+$Comp
+L +5V #PWR?
+U 1 1 4EE3787E
+P 4200 6500
+F 0 "#PWR?" H 4200 6590 20  0001 C CNN
+F 1 "+5V" H 4200 6590 30  0000 C CNN
+	1    4200 6500
+	-1   0    0    1
+$EndComp
+Text Label 4300 6500 3    60   ~ 0
+Arduino - SCL
+Text Label 4000 6500 3    60   ~ 0
+Arduino - SDA
+$Comp
+L CONN_4 P?
+U 1 1 4EE37809
+P 4150 6050
+F 0 "P?" V 4100 6050 50  0000 C CNN
+F 1 "CONN_4" V 4200 6050 50  0000 C CNN
+	1    4150 6050
+	0    -1   -1   0
+$EndComp
 $Comp
 L +5V #PWR?
 U 1 1 4EE364FB
 P 2300 4850
-F 0 "#PWR?" H 2300 4940 20  0001 C C
-F 1 "+5V" H 2300 4940 30  0000 C C
+F 0 "#PWR?" H 2300 4940 20  0001 C CNN
+F 1 "+5V" H 2300 4940 30  0000 C CNN
 	1    2300 4850
 	-1   0    0    1
@@
 U 1 1 4EE364FA
 P 2200 4400
-F 0 "P?" V 2150 4400 40  0000 C C
-F 1 "CONN_2" V 2250 4400 40  0000 C C
+F 0 "P?" V 2150 4400 40  0000 C CNN
+F 1 "CONN_2" V 2250 4400 40  0000 C CNN
 	1    2200 4400
 	0    -1   -1   0
 $EndComp
-Text Label 2100 5500 3    60   ~
+Text Label 2100 5500 3    60   ~ 0
 Arduino - Pression exterieure
 $Comp
@@
 U 1 1 4EE364F9
 P 2100 5100
-F 0 "R?" V 2180 5100 50  0000 C C
-F 1 "R" V 2100 5100 50  0000 C C
+F 0 "R?" V 2180 5100 50  0000 C CNN
+F 1 "R" V 2100 5100 50  0000 C CNN
 	1    2100 5100
 	1    0    0    -1
@@
 U 1 1 4EE364F8
 P 1700 5100
-F 0 "R?" V 1780 5100 50  0000 C C
-F 1 "R" V 1700 5100 50  0000 C C
+F 0 "R?" V 1780 5100 50  0000 C CNN
+F 1 "R" V 1700 5100 50  0000 C CNN
 	1    1700 5100
 	1    0    0    -1
 $EndComp
-Text Label 1700 5500 3    60   ~
+Text Label 1700 5500 3    60   ~ 0
 Arduino - Temperature exterieure
 $Comp
@@
 U 1 1 4EE364F7
 P 1800 4400
-F 0 "P?" V 1750 4400 40  0000 C C
-F 1 "CONN_2" V 1850 4400 40  0000 C C
+F 0 "P?" V 1750 4400 40  0000 C CNN
+F 1 "CONN_2" V 1850 4400 40  0000 C CNN
 	1    1800 4400
 	0    -1   -1   0
@@
 U 1 1 4EE364F6
 P 1900 4850
-F 0 "#PWR?" H 1900 4940 20  0001 C C
-F 1 "+5V" H 1900 4940 30  0000 C C
+F 0 "#PWR?" H 1900 4940 20  0001 C CNN
+F 1 "+5V" H 1900 4940 30  0000 C CNN
 	1    1900 4850
 	-1   0    0    1
 $EndComp
-Wire Wire Line
-	1300 5350 1300 5500
-Wire Wire Line
-	1300 4750 1300 4850
-Wire Wire Line
-	1500 4850 1500 4750
-Wire Wire Line
-	1100 4850 1100 4750
-Wire Wire Line
-	900  4750 900  4850
-Wire Wire Line
-	900  5350 900  5500
 $Comp
 L +5V #PWR?
 U 1 1 4EE22ACD
 P 1500 4850
-F 0 "#PWR?" H 1500 4940 20  0001 C C
-F 1 "+5V" H 1500 4940 30  0000 C C
+F 0 "#PWR?" H 1500 4940 20  0001 C CNN
+F 1 "+5V" H 1500 4940 30  0000 C CNN
 	1    1500 4850
 	-1   0    0    1
@@
 U 1 1 4EE22ACC
 P 1400 4400
-F 0 "P?" V 1350 4400 40  0000 C C
-F 1 "CONN_2" V 1450 4400 40  0000 C C
+F 0 "P?" V 1350 4400 40  0000 C CNN
+F 1 "CONN_2" V 1450 4400 40  0000 C CNN
 	1    1400 4400
 	0    -1   -1   0
 $EndComp
-Text Label 1300 5500 3    60   ~
+Text Label 1300 5500 3    60   ~ 0
 Arduino - Pression interieure
 $Comp
@@
 U 1 1 4EE22ACB
 P 1300 5100
-F 0 "R?" V 1380 5100 50  0000 C C
-F 1 "R" V 1300 5100 50  0000 C C
+F 0 "R?" V 1380 5100 50  0000 C CNN
+F 1 "R" V 1300 5100 50  0000 C CNN
 	1    1300 5100
 	1    0    0    -1
@@
 U 1 1 4EE1ADE8
 P 900 5100
-F 0 "R?" V 980 5100 50  0000 C C
-F 1 "R" V 900 5100 50  0000 C C
+F 0 "R?" V 980 5100 50  0000 C CNN
+F 1 "R" V 900 5100 50  0000 C CNN
 	1    900  5100
 	1    0    0    -1
 $EndComp
-Text Label 900  5500 3    60   ~
+Text Label 900  5500 3    60   ~ 0
 Arduino - Temperature interieure
 $Comp
@@
 U 1 1 4EE1AD34
 P 1000 4400
-F 0 "P?" V 950 4400 40  0000 C C
-F 1 "CONN_2" V 1050 4400 40  0000 C C
+F 0 "P?" V 950 4400 40  0000 C CNN
+F 1 "CONN_2" V 1050 4400 40  0000 C CNN
 	1    1000 4400
 	0    -1   -1   0
@@
 U 1 1 4EE0BB2B
 P 1100 4850
-F 0 "#PWR?" H 1100 4940 20  0001 C C
-F 1 "+5V" H 1100 4940 30  0000 C C
+F 0 "#PWR?" H 1100 4940 20  0001 C CNN
+F 1 "+5V" H 1100 4940 30  0000 C CNN
 	1    1100 4850
 	-1   0    0    1
