File: Electronique/Pression/pression.sch (KiCad schematic (older format))
At the start: 15 parts

Commit message: Modifications de la shield pour les capteurs
Parts:
- added 10k, 10k?, CAPT_TEMP, CAPT_TEMP?: R, symbol R
- added GND: VSS, symbol VSS
- added SHIELD?: ARDUINO_SHIELD, symbol ARDUINO_SHIELD
- gave numbers to parts that had none: 1
- renumbered +9V to +9V05, +9V to +9V07, GND to GND06, GND to GND08, MPX~2200AP to MPX~2200AP1, POT to POT1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
Connections:
- net labels added: Entree temperature ext, Entree temperature int, VCC
- wire segments 33 -> 41
