File: Electronique/Modulation FSK/Carte/Shield FSK.sch (KiCad schematic (older format))
At the start: 15 parts, among them P1 BNC, P2 CONN_2, U1 XR2206, U2 LM7810

Commit message: maj du schématique du Shield FSK.
Parts:
- added C5, C6: CP, symbol CP
- added D1: DIODE, symbol DIODE
- added D2: LED, symbol LED
- added L1, L2: INDUCTOR, symbol INDUCTOR
- added P3: CONN_2, symbol CONN_2
- added R6, R7: R, symbol R
Connections:
- net labels removed: +BATT
- wire segments 44 -> 67
- no-connect marks 28 -> 27
Other:
- moved on the sheet: C1, C2, C3, C4, P1, P2, R1, R2, R3, R4, R5, RV1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
